File: ljhs-1.kicad_pcb (KiCad board)
At the start: 2 copper layers, 75 x 54 mm, 32 parts, among them P1 Digital, P2 Analog, P3 CONN_1, P4 CONN_1, P5 CONN_1, P6 CONN_1, P7 IR_RECVR, P8 PWR, P9 LDR, Q1 Q_NMOS_GSD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

Commit message: Routing complete.
Routing:
- net +5V: track 0.00 -> 163.2 mm
- net /3(**): track 0.00 -> 71.2 mm, vias 0 -> 2
- net /6(**): track 0.00 -> 43.7 mm, vias 0 -> 1
- net /11(**/MISO): track 0.00 -> 37.4 mm, vias 0 -> 1
- net /5(**): track 0.00 -> 36.4 mm, vias 0 -> 1
- net /A0: track 0.00 -> 25.3 mm
- net Net-(D7-Pad2): track 0.00 -> 19.9 mm, vias 0 -> 1
- net /Vin: track 0.00 -> 17.0 mm
- net /7: track 0.00 -> 14.6 mm, vias 0 -> 1
- net /8: track 0.00 -> 12.7 mm
- net Net-(D6-Pad1): track 0.00 -> 7.10 mm, vias 0 -> 1
- net Net-(D5-Pad1): track 0.00 -> 7.10 mm, vias 0 -> 1
- net /4: track 0.00 -> 6.65 mm
- net Net-(Q2-Pad3): track 0.00 -> 4.52 mm
- net Net-(Q1-Pad3): track 0.00 -> 4.52 mm
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- added copper zone on B.Cu, net GND
- added copper zone on F.Cu, net GND
