File: v2kicad/v2kicad.kicad_pcb (KiCad board)
At the start: 2 copper layers, 3 parts

Commit message: Progress
Parts:
- added REF**: MountingHole_3.2mm_M3, Mounting_Holes:MountingHole_3.2mm_M3, F.Cu at (163.0, 78.0)
- BT1: footprint xxx:CR2032-white-smd -> sydcon-badges-2016:CR2032-white-smd (1); moved to B.Cu
- R1: moved to B.Cu
- moved D1 48.7 mm to (184.6, 107.7), turned to 41.5 degrees
- moved BT1 35.8 mm to (163.0, 116.0)
- moved R1 12.2 mm to (163.0, 107.0), turned to 180 degrees
Other:
- board outline added: 72 x 59 mm
- rule pad_to_mask_clearance: 0.2 -> 0
- board text added: "#letsjusthackshit"
- board text added: "A drinking club with a hacking problem"
- board text added: "CON"
- board text added: "PLATYPUS"
